File: kicad/chouchou.kicad_pcb (KiCad board)
At the start: 2 copper layers, 206.6 x 122 mm, 21 parts

Commit message: add wiring
Parts:
- added S21: , PG1350, F.Cu at (36.6, 136.6)
- added S22: , PG1350, F.Cu at (41.0, 120.2)
- added S23: , PG1350, F.Cu at (60.9, 134.8)
- added S24: , PG1350, F.Cu at (68.1, 119.4)
- added S25: , PG1350, F.Cu at (82.0, 139.2)
- added S26: , PG1350, F.Cu at (90.5, 124.4)
- added S27: , PG1350, F.Cu at (98.0, 157.6)
- added S28: , PG1350, F.Cu at (107.7, 143.7)
- added S29: , PG1350, F.Cu at (82.8, 200.6)
- added S30: , PG1350, F.Cu at (96.9, 211.7)
- added S31: , PG1350, F.Cu at (223.8, 136.6)
- added S32: , PG1350, F.Cu at (219.4, 120.2)
- added S33: , PG1350, F.Cu at (199.5, 134.8)
- added S34: , PG1350, F.Cu at (192.3, 119.4)
- added S35: , PG1350, F.Cu at (178.4, 139.2)
- added S36: , PG1350, F.Cu at (169.9, 124.4)
- added S37: , PG1350, F.Cu at (162.5, 157.6)
- added S38: , PG1350, F.Cu at (152.7, 143.7)
- added S39: , PG1350, F.Cu at (177.7, 200.6)
- added S40: , PG1350, F.Cu at (163.5, 211.7)
- moved S12 5.80 mm to (219.4, 120.2), turned to 15 degrees
- moved S11 5.80 mm to (223.8, 136.6), turned to 15 degrees
- moved S6 3.00 mm to (90.5, 124.4), turned to -30 degrees
- moved S19 3.00 mm to (177.7, 200.6), turned to -52 degrees
- moved S5 3.00 mm to (82.0, 139.2), turned to -30 degrees
- moved S17 3.00 mm to (162.5, 157.6), turned to 35 degrees
- moved S3 3.00 mm to (60.9, 134.8), turned to -25 degrees
- moved S10 3.00 mm to (96.9, 211.7), turned to 52 degrees
- moved S7 3.00 mm to (98.0, 157.6), turned to -35 degrees
- moved S13 3.00 mm to (199.5, 134.8), turned to 25 degrees
- moved S9 3.00 mm to (82.8, 200.6), turned to 52 degrees
- moved S16 3.00 mm to (169.9, 124.4), turned to 30 degrees
- moved S20 3.00 mm to (163.5, 211.7), turned to -52 degrees
- moved S15 3.00 mm to (178.4, 139.2), turned to 30 degrees
- moved S18 3.00 mm to (152.7, 143.7), turned to 35 degrees
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Routing:
- net GND: track 0.00 -> 774.7 mm
- net GP12: track 0.00 -> 121.3 mm
- net GP26: track 0.00 -> 119.9 mm
- net GP7: track 0.00 -> 103.6 mm
- net GP3: track 0.00 -> 101.1 mm
- net GP13: track 0.00 -> 96.7 mm
- net GP27: track 0.00 -> 92.7 mm
- net GP6: track 0.00 -> 81.8 mm
- net GP10: track 0.00 -> 80.0 mm
- net GP2: track 0.00 -> 76.2 mm
- net GP11: track 0.00 -> 75.2 mm
- net GP14: track 0.00 -> 70.9 mm
- net GP5: track 0.00 -> 69.0 mm
- net GP28: track 0.00 -> 65.3 mm
- net GP9: track 0.00 -> 64.5 mm
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Other:
- board size 206.6 x 122 mm -> 212.4 x 122 mm
- net class Default removed

Commit message: Update design
Parts:
- moved S10 76.8 mm to (127.4, 141.2), turned to 58 degrees
- moved S30 76.8 mm to (127.4, 141.2), turned to -122 degrees
- moved S29 75.0 mm to (112.1, 131.6), turned to -122 degrees
- moved S9 75.0 mm to (112.1, 131.6), turned to 58 degrees
- moved S20 71.4 mm to (174.5, 141.2), turned to -58 degrees
- moved S40 71.4 mm to (174.5, 141.2), turned to 122 degrees
- moved S19 70.0 mm to (189.7, 131.6), turned to -58 degrees
- moved S39 70.0 mm to (189.7, 131.6), turned to 122 degrees
- moved RP2040Zero1 66.1 mm to (140.9, 104.9)
- moved S28 66.1 mm to (128.4, 80.9)
- moved S8 66.1 mm to (128.4, 80.9)
- moved S1 66.1 mm to (57.3, 73.8)
- moved S11 66.1 mm to (244.5, 73.8)
- moved S12 66.1 mm to (240.1, 57.4)
- moved S18 66.1 mm to (173.4, 80.9)
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Routing:
- net GND: track 774.7 -> 840.4 mm
- net GP9: track 64.5 -> 52.3 mm
- net GP10: track 80.0 -> 68.0 mm
- net GP8: track 58.5 -> 48.3 mm
- net GP11: track 75.2 -> 66.0 mm
- net GP27: track 92.7 -> 89.0 mm
- net GP26: track 119.9 -> 116.8 mm
- net GP15: track 43.9 -> 46.9 mm
- net GP5: track 69.0 -> 66.3 mm
- net GP13: track 96.7 -> 95.2 mm
- net GP2: track 76.2 -> 75.0 mm
- net GP1: track 56.6 -> 55.4 mm
- net GP28: track 65.3 -> 64.4 mm
- net GP3: track 101.1 -> 100.4 mm
- net GP4: track 37.3 -> 36.8 mm
Other:
- board size 212.4 x 122 mm -> 212.4 x 114.4 mm

Commit message: Add images
Parts:
- added ?: LOGO, images:蝶, F.Cu at (91.7, 98.5)
- added ?: LOGO, images:々, F.Cu at (213.7, 95.9)
- added G***: LOGO, images:butterfly, F.Cu at (153.3, 113.5)
- added _1: , MountingHole_2.2mm_M2_Pad_Via, F.Cu at (79.2, 47.8)
- added _2: , MountingHole_2.2mm_M2_Pad_Via, F.Cu at (67.7, 90.7)
- added _3: , MountingHole_2.2mm_M2_Pad_Via, F.Cu at (227.5, 47.8)
- added _4: , MountingHole_2.2mm_M2_Pad_Via, F.Cu at (239.1, 90.7)
- added _5: , MountingHole_2.2mm_M2_Pad_Via, F.Cu at (153.4, 117.1)
- moved S11 4.51 mm to (247.0, 70.0)
- moved S31 4.51 mm to (247.0, 70.0)
- moved S20 4.51 mm to (176.9, 137.4)
- moved S40 4.51 mm to (176.9, 137.4)
- moved S27 4.51 mm to (121.1, 91.0)
- moved S7 4.51 mm to (121.1, 91.0)
- moved S12 4.51 mm to (242.6, 53.6)
- moved S16 4.51 mm to (193.0, 57.8)
- moved S2 4.51 mm to (64.2, 53.6)
- moved S22 4.51 mm to (64.2, 53.6)
- moved S26 4.51 mm to (113.7, 57.8)
- moved S32 4.51 mm to (242.6, 53.6)
- moved S36 4.51 mm to (193.0, 57.8)
- moved S6 4.51 mm to (113.7, 57.8)
- moved S10 4.51 mm to (129.8, 137.4)
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Routing:
- net GND: track 840.4 -> 808.7 mm
- net GP11: track 66.0 -> 63.4 mm
- net GP26: track 116.8 -> 118.7 mm
- net GP5: track 66.3 -> 65.4 mm

Commit message: Add ordered files
Parts:
- removed the ? at (91.7, 98.5)
- removed the ? at (213.7, 95.9)
- removed G***: LOGO, images:butterfly
- added ?: LOGO, images:butterfly_right, F.Cu at (168.7, 108.7)
- added ?: LOGO, images:butterfly_left, F.Cu at (133.2, 108.7)
- added _6: , MountingHole_2.2mm_M2_Pad_Via, F.Cu at (178.5, 60.6)
- added _7: , MountingHole_2.2mm_M2_Pad_Via, F.Cu at (114.1, 142.9)
- added _8: , MountingHole_2.2mm_M2_Pad_Via, F.Cu at (189.1, 142.9)
- moved _2 163.9 mm to (225.0, 44.9), turned to 15 degrees
- moved _3 135.1 mm to (97.2, 83.4), turned to -30 degrees
- moved _5 63.2 mm to (124.8, 60.6), turned to -35 degrees
- moved _4 33.8 mm to (206.0, 83.4), turned to 30 degrees
- moved _1 3.00 mm to (78.2, 44.9)
- moved RP2040Zero1 1.74 mm to (141.6, 101.1)
- moved S11 1.74 mm to (245.2, 70.0)
- moved S12 1.74 mm to (240.8, 53.6)
- moved S14 1.74 mm to (213.7, 52.9)
- moved S17 1.74 mm to (183.9, 91.0)
- moved S18 1.74 mm to (174.1, 77.1)
- moved S19 1.74 mm to (190.4, 127.9)
- moved S27 1.74 mm to (119.4, 91.0)
- moved S28 1.74 mm to (129.1, 77.1)
- moved S29 1.74 mm to (112.8, 127.9)
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Routing:
- net GND: track 808.7 -> 819.8 mm
- net GP12: track 121.3 -> 129.0 mm
- net GP7: track 103.6 -> 105.8 mm
- net GP13: track 95.2 -> 97.2 mm
- net GP26: track 118.7 -> 120.5 mm
- net GP2: track 75.3 -> 76.1 mm
- net GP11: track 63.4 -> 64.0 mm
Other:
- board size 212.4 x 114.4 mm -> 210.5 x 114.4 mm

Commit message: Connect pcb
Parts:
- removed ?: LOGO, images:butterfly_right
- removed ?: LOGO, images:butterfly_left
- added RP2040Zero2: , RP2040-Zero, F.Cu at (158.3, 78.8)
- added S41, S58: , PG1350, F.Cu at (227.4, 67.1)
- added S42, S59: , PG1350, F.Cu at (227.4, 50.1)
- added S43, S60: , PG1350, F.Cu at (227.4, 33.1)
- added S44, S61: , PG1350, F.Cu at (209.2, 72.7)
- added S45, S62: , PG1350, F.Cu at (208.3, 55.7)
- added S46, S63: , PG1350, F.Cu at (207.4, 38.7)
- added S47, S64: , PG1350, F.Cu at (191.4, 77.0)
- added S48, S65: , PG1350, F.Cu at (190.5, 60.0)
- added S49, S66: , PG1350, F.Cu at (189.6, 43.1)
- added S50, S67: , PG1350, F.Cu at (203.4, 100.2)
- added S51, S68: , PG1350, F.Cu at (183.4, 105.0)
- added S52: , PG1350, F.Cu at (264.8, 80.0)
- added S53: , PG1350, F.Cu at (266.3, 63.1)
- added S54: , PG1350, F.Cu at (267.8, 46.1)
- added S55: , PG1350, F.Cu at (245.4, 72.7)
- added S56: , PG1350, F.Cu at (245.4, 55.7)
- added S57: , PG1350, F.Cu at (245.4, 38.7)
- added TRRS1: TRRS-PJ-320A-dual, TRRS-PJ-320A-dual, F.Cu at (138.0, 86.1)
- added TRRS2: TRRS-PJ-320A-dual, TRRS-PJ-320A-dual, F.Cu at (156.8, 81.6)
- moved S19 174.4 mm to (28.5, 63.1), turned to -175 degrees
- moved S20 174.0 mm to (27.0, 46.1), turned to -175 degrees
- moved _2 161.2 mm to (67.4, 79.1), turned to 0 degrees
- moved S11 159.3 mm to (86.5, 55.7), turned to -3 degrees
- moved S12 154.1 mm to (87.4, 38.7), turned to -3 degrees
- moved _7 152.9 mm to (214.0, 27.2), turned to 3 degrees
- moved S18 144.1 mm to (30.0, 80.0), turned to -175 degrees
- moved S31 141.3 mm to (104.3, 60.0), turned to 177 degrees
- moved _5 136.7 mm to (258.8, 33.8), turned to -5 degrees
- moved S32 136.0 mm to (105.2, 43.1), turned to 177 degrees
- moved S33 133.4 mm to (91.4, 100.2), turned to -96 degrees
- moved S40 121.2 mm to (245.4, 38.7), turned to 0 degrees
- moved S13 117.8 mm to (103.4, 77.0), turned to -3 degrees
- moved S34 114.9 mm to (111.4, 105.0), turned to -111 degrees
- moved _4 111.2 mm to (98.8, 112.8), turned to 69 degrees
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Connections:
- RP2040Zero1 pad 10: GP9 -> matrix_outer_bottom
- RP2040Zero1 pad 11: GP10 -> matrix_pinky_middle
- RP2040Zero1 pad 12: GP11 -> matrix_ring_middle
- RP2040Zero1 pad 13: GP12 -> matrix_middle_middle
- RP2040Zero1 pad 14: GP13 -> matrix_index_middle
- RP2040Zero1 pad 15: GP14 -> matrix_outer_middle
- RP2040Zero1 pad 16: GP15 -> matrix_pinky_top
- RP2040Zero1 pad 17: GP26 -> matrix_ring_top
- RP2040Zero1 pad 18: GP27 -> matrix_middle_top
- RP2040Zero1 pad 2: GP1 -> SCL
- RP2040Zero1 pad 22: GP28 -> matrix_index_top
- RP2040Zero1 pad 23: GP29 -> matrix_outer_top
- RP2040Zero1 pad 4: GP3 -> thumbs_outer_cluster
- RP2040Zero1 pad 5: GP4 -> thumbs_inner_cluster
- RP2040Zero1 pad 6: GP5 -> matrix_pinky_bottom
- RP2040Zero1 pad 7: GP6 -> matrix_ring_bottom
- RP2040Zero1 pad 8: GP7 -> matrix_middle_bottom
- RP2040Zero1 pad 9: GP8 -> matrix_index_bottom
- S1 pad 1: GP12 -> matrix_pinky_bottom
- S10 pad 1: GP10 -> matrix_index_bottom
- S11 pad 1: GP7 -> matrix_index_middle
- S12 pad 1: GP3 -> matrix_index_top
- S13 pad 1: GP6 -> matrix_outer_bottom
- S14 pad 1: GP2 -> matrix_outer_middle
- S15 pad 1: GP5 -> matrix_outer_top
- S16 pad 1: GP1 -> thumbs_inner_cluster
- S17 pad 1: GP4 -> thumbs_outer_cluster
- S18 pad 1: GP0 -> matrix_pinky_bottom
- S19 pad 1: GP8 -> matrix_pinky_middle
- S2 pad 1: GP26 -> matrix_pinky_middle
- S20 pad 1: GP9 -> matrix_pinky_top
- S21 pad 1: GP12 -> matrix_ring_bottom
- S22 pad 1: GP26 -> matrix_ring_middle
- S23 pad 1: GP13 -> matrix_ring_top
- S24 pad 1: GP27 -> matrix_middle_bottom
- S25 pad 1: GP14 -> matrix_middle_middle
- S26 pad 1: GP28 -> matrix_middle_top
- S27 pad 1: GP15 -> matrix_index_bottom
- S28 pad 1: GP29 -> matrix_index_middle
- S29 pad 1: GP11 -> matrix_index_top
- S3 pad 1: GP13 -> matrix_pinky_top
- S30 pad 1: GP10 -> matrix_outer_bottom
- S31 pad 1: GP7 -> matrix_outer_middle
- S32 pad 1: GP3 -> matrix_outer_top
- S33 pad 1: GP6 -> thumbs_inner_cluster
- S34 pad 1: GP2 -> thumbs_outer_cluster
- S35 pad 1: GP5 -> mirror_matrix_pinky_bottom
- S35 pad 2: GND -> rGND
- S36 pad 1: GP1 -> mirror_matrix_pinky_middle
- S36 pad 2: GND -> rGND
- S37 pad 1: GP4 -> mirror_matrix_pinky_top
- S37 pad 2: GND -> rGND
- S38 pad 1: GP0 -> mirror_matrix_ring_bottom
- S38 pad 2: GND -> rGND
- S39 pad 1: GP8 -> mirror_matrix_ring_middle
- S39 pad 2: GND -> rGND
- S4 pad 1: GP27 -> matrix_ring_bottom
- S40 pad 1: GP9 -> mirror_matrix_ring_top
- S40 pad 2: GND -> rGND
- S5 pad 1: GP14 -> matrix_ring_middle
- S6 pad 1: GP28 -> matrix_ring_top
- S7 pad 1: GP15 -> matrix_middle_bottom
- S8 pad 1: GP29 -> matrix_middle_middle
- S9 pad 1: GP11 -> matrix_middle_top
Routing:
- net rGND: track 0.00 -> 522.7 mm
- net GND: track 819.8 -> 444.7 mm
- net matrix_pinky_bottom: track 0.00 -> 144.9 mm
- net matrix_pinky_top: track 0.00 -> 132.7 mm
- net matrix_pinky_middle: track 0.00 -> 132.1 mm
- net GP12: track 129.0 -> 0.00 mm
- net matrix_ring_bottom: track 0.00 -> 122.3 mm
- net GP26: track 120.5 -> 0.00 mm
- net mirror_matrix_pinky_middle: track 0.00 -> 115.4 mm
- net mirror_matrix_pinky_bottom: track 0.00 -> 114.1 mm
- net mirror_matrix_pinky_top: track 0.00 -> 111.4 mm
- net matrix_ring_middle: track 0.00 -> 108.9 mm
- net matrix_ring_top: track 0.00 -> 106.8 mm
- net GP7: track 105.8 -> 0.00 mm
- net GP3: track 100.8 -> 0.00 mm
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Other:
- board size 210.5 x 114.4 mm -> 262.1 x 95.9 mm

Commit message: Cleanup tracks
Routing:
- net GND: track 444.7 -> 460.6 mm
- net mirror_matrix_pinky_bottom: track 114.1 -> 124.7 mm
- net mirror_matrix_ring_middle: track 87.6 -> 83.1 mm
- net mirror_matrix_pinky_middle: track 115.4 -> 111.1 mm
- net mirror_matrix_ring_bottom: track 98.1 -> 95.6 mm
- net matrix_ring_bottom: track 122.3 -> 120.3 mm
- net matrix_index_middle: track 68.0 -> 66.2 mm
- net matrix_ring_middle: track 108.9 -> 107.2 mm
- net mirror_matrix_index_middle: track 44.0 -> 42.5 mm
- net mirror_matrix_index_top: track 44.9 -> 43.4 mm
- net mirror_matrix_middle_middle: track 66.5 -> 65.1 mm
- net matrix_middle_bottom: track 100.5 -> 99.3 mm
- net mirror_matrix_middle_top: track 67.9 -> 66.8 mm
- net matrix_index_bottom: track 72.0 -> 70.9 mm
- net matrix_middle_middle: track 89.0 -> 90.1 mm
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
Commit message: Add traces
Parts:
- added S69: , PG1350, F.Cu at (189.0, 44.8)
- added S70: , PG1350, F.Cu at (216.2, 101.6)
- added S71: , PG1350, F.Cu at (194.6, 98.2)
- added S72: , PG1350, F.Cu at (173.4, 102.3)
- moved S35 166.7 mm to (99.1, 98.2), turned to 178 degrees
- moved S36 151.3 mm to (120.2, 102.3), turned to 160 degrees
- moved S54 109.8 mm to (173.4, 102.3), turned to 20 degrees
- moved S18 92.9 mm to (120.2, 102.3), turned to -20 degrees
- moved S53 79.9 mm to (194.6, 98.2), turned to 2 degrees
- moved _3 61.5 mm to (77.0, 88.5), turned to 18 degrees
- moved _7 61.4 mm to (216.6, 88.5), turned to -18 degrees
- moved S51 60.5 mm to (189.0, 44.8), turned to 2 degrees
- moved S33 57.0 mm to (104.7, 44.8), turned to 178 degrees
- moved S52 53.3 mm to (216.2, 101.6), turned to -18 degrees
- moved _6 52.7 mm to (212.4, 28.5), turned to 2 degrees
- moved _2 52.4 mm to (81.2, 28.5), turned to -2 degrees
- moved S68 43.7 mm to (189.5, 61.7), turned to -178 degrees
- moved S27 43.6 mm to (67.4, 33.1), turned to 180 degrees
- moved S50 40.9 mm to (189.5, 61.7), turned to 2 degrees
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Connections:
- RP2040Zero1 pad 3: GP2 -> thumbs_outer_cluster
- RP2040Zero1 pad 4: thumbs_outer_cluster -> thumbs_middle_cluster
- RP2040Zero2 pad 1: mirror_matrix_outer_top -> rGND
- RP2040Zero2 pad 10: mirror_matrix_pinky_middle -> mirror_matrix_middle_middle
- RP2040Zero2 pad 11: mirror_matrix_outer_bottom -> mirror_matrix_ring_middle
- RP2040Zero2 pad 12: mirror_matrix_index_bottom -> mirror_matrix_pinky_middle
- RP2040Zero2 pad 13: mirror_matrix_middle_bottom -> mirror_matrix_outer_bottom
- RP2040Zero2 pad 14: mirror_matrix_ring_bottom -> mirror_matrix_index_bottom
- RP2040Zero2 pad 15: mirror_matrix_pinky_bottom -> mirror_matrix_middle_bottom
- RP2040Zero2 pad 16: mirror_thumbs_inner_cluster -> mirror_matrix_ring_bottom
- RP2040Zero2 pad 17: mirror_thumbs_outer_cluster -> mirror_matrix_pinky_bottom
- RP2040Zero2 pad 18: rSCL -> mirror_thumbs_inner_cluster
- RP2040Zero2 pad 2: mirror_matrix_index_top -> rSCL
- RP2040Zero2 pad 22: rGP28 -> mirror_thumbs_middle_cluster
- RP2040Zero2 pad 23: rGND -> mirror_thumbs_outer_cluster
- RP2040Zero2 pad 3: mirror_matrix_middle_top -> mirror_matrix_outer_top
- RP2040Zero2 pad 4: mirror_matrix_ring_top -> mirror_matrix_index_top
- RP2040Zero2 pad 5: mirror_matrix_pinky_top -> mirror_matrix_middle_top
- RP2040Zero2 pad 6: mirror_matrix_outer_middle -> mirror_matrix_ring_top
- RP2040Zero2 pad 7: mirror_matrix_index_middle -> mirror_matrix_pinky_top
- RP2040Zero2 pad 8: mirror_matrix_middle_middle -> mirror_matrix_outer_middle
- RP2040Zero2 pad 9: mirror_matrix_ring_middle -> mirror_matrix_index_middle
- S17 pad 1: thumbs_outer_cluster -> thumbs_middle_cluster
- S18 pad 1: matrix_pinky_bottom -> thumbs_outer_cluster
- S19 pad 1: matrix_pinky_middle -> matrix_pinky_bottom
- S20 pad 1: matrix_pinky_top -> matrix_pinky_middle
- S21 pad 1: matrix_ring_bottom -> matrix_pinky_top
- S22 pad 1: matrix_ring_middle -> matrix_ring_bottom
- S23 pad 1: matrix_ring_top -> matrix_ring_middle
- S24 pad 1: matrix_middle_bottom -> matrix_ring_top
- S25 pad 1: matrix_middle_middle -> matrix_middle_bottom
- S26 pad 1: matrix_middle_top -> matrix_middle_middle
- S27 pad 1: matrix_index_bottom -> matrix_middle_top
- S28 pad 1: matrix_index_middle -> matrix_index_bottom
- S29 pad 1: matrix_index_top -> matrix_index_middle
- S30 pad 1: matrix_outer_bottom -> matrix_index_top
- S31 pad 1: matrix_outer_middle -> matrix_outer_bottom
- S32 pad 1: matrix_outer_top -> matrix_outer_middle
- S33 pad 1: thumbs_inner_cluster -> matrix_outer_top
- S34 pad 1: thumbs_outer_cluster -> thumbs_inner_cluster
- S35 pad 1: mirror_matrix_pinky_bottom -> thumbs_middle_cluster
- S35 pad 2: rGND -> GND
- S36 pad 1: mirror_matrix_pinky_middle -> thumbs_outer_cluster
- S36 pad 2: rGND -> GND
- S37 pad 1: mirror_matrix_pinky_top -> mirror_matrix_pinky_bottom
- S38 pad 1: mirror_matrix_ring_bottom -> mirror_matrix_pinky_middle
- S39 pad 1: mirror_matrix_ring_middle -> mirror_matrix_pinky_top
- S40 pad 1: mirror_matrix_ring_top -> mirror_matrix_ring_bottom
- S41 pad 1: mirror_matrix_middle_bottom -> mirror_matrix_ring_middle
- S42 pad 1: mirror_matrix_middle_middle -> mirror_matrix_ring_top
- S43 pad 1: mirror_matrix_middle_top -> mirror_matrix_middle_bottom
- S44 pad 1: mirror_matrix_index_bottom -> mirror_matrix_middle_middle
- S45 pad 1: mirror_matrix_index_middle -> mirror_matrix_middle_top
- S46 pad 1: mirror_matrix_index_top -> mirror_matrix_index_bottom
- S47 pad 1: mirror_matrix_outer_bottom -> mirror_matrix_index_middle
- S48 pad 1: mirror_matrix_outer_middle -> mirror_matrix_index_top
- S49 pad 1: mirror_matrix_outer_top -> mirror_matrix_outer_bottom
- S50 pad 1: mirror_thumbs_inner_cluster -> mirror_matrix_outer_middle
- S51 pad 1: mirror_thumbs_outer_cluster -> mirror_matrix_outer_top
- S52 pad 1: mirror_matrix_pinky_bottom -> mirror_thumbs_inner_cluster
- S53 pad 1: mirror_matrix_pinky_middle -> mirror_thumbs_middle_cluster
- S54 pad 1: mirror_matrix_pinky_top -> mirror_thumbs_outer_cluster
- S55 pad 1: mirror_matrix_ring_bottom -> mirror_matrix_pinky_bottom
- S56 pad 1: mirror_matrix_ring_middle -> mirror_matrix_pinky_middle
- S57 pad 1: mirror_matrix_ring_top -> mirror_matrix_pinky_top
- S58 pad 1: mirror_matrix_middle_bottom -> mirror_matrix_ring_bottom
- S59 pad 1: mirror_matrix_middle_middle -> mirror_matrix_ring_middle
- S60 pad 1: mirror_matrix_middle_top -> mirror_matrix_ring_top
- S61 pad 1: mirror_matrix_index_bottom -> mirror_matrix_middle_bottom
- S62 pad 1: mirror_matrix_index_middle -> mirror_matrix_middle_middle
- S63 pad 1: mirror_matrix_index_top -> mirror_matrix_middle_top
- S64 pad 1: mirror_matrix_outer_bottom -> mirror_matrix_index_bottom
- S65 pad 1: mirror_matrix_outer_middle -> mirror_matrix_index_middle
- S66 pad 1: mirror_matrix_outer_top -> mirror_matrix_index_top
- S67 pad 1: mirror_thumbs_inner_cluster -> mirror_matrix_outer_bottom
- S68 pad 1: mirror_thumbs_outer_cluster -> mirror_matrix_outer_middle
Routing:
- net thumbs_middle_cluster: track 0.00 -> 74.9 mm
- net mirror_thumbs_middle_cluster: track 0.00 -> 64.4 mm
- net GND: track 460.6 -> 501.2 mm
- net mirror_thumbs_inner_cluster: track 66.0 -> 95.1 mm
- net rSCL: track 16.6 -> 44.1 mm
- net thumbs_inner_cluster: track 83.1 -> 107.9 mm
- net thumbs_outer_cluster: track 70.3 -> 55.4 mm
- net matrix_pinky_middle: track 132.2 -> 124.2 mm
- net mirror_matrix_ring_bottom: track 95.6 -> 103.4 mm
- net mirror_thumbs_outer_cluster: track 51.5 -> 59.0 mm
- net matrix_index_middle: track 66.2 -> 59.4 mm
- net matrix_middle_middle: track 90.1 -> 83.5 mm
- net mirror_matrix_ring_middle: track 83.1 -> 88.8 mm
- net matrix_pinky_top: track 132.7 -> 127.1 mm
- net mirror_matrix_outer_bottom: track 28.1 -> 33.5 mm
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Other:
- board size 262.1 x 95.9 mm -> 261 x 90.8 mm

Commit message: use full duplex serial
Connections:
- net SCL renamed RX
- RP2040Zero1 pad 1: GP0 -> TX
- RP2040Zero2 pad 1: rGND -> rTX
- RP2040Zero2 pad 2: rSCL -> rRX
- TRRS1 pad 4: D -> TX
- TRRS2 pad 3: rSCL -> rTX
- TRRS2 pad 4: rD -> rRX
Routing:
- net rSCL: track 44.1 -> 0.00 mm
- net rTX: track 0.00 -> 44.0 mm
- net rRX: track 0.00 -> 43.2 mm
- net TX: track 0.00 -> 33.4 mm
- net mirror_thumbs_middle_cluster: track 64.4 -> 73.6 mm
- net rP3V3: track 29.6 -> 37.9 mm
- net mirror_thumbs_outer_cluster: track 59.0 -> 64.3 mm
- net mirror_thumbs_inner_cluster: track 95.1 -> 92.5 mm
- net rGND: track 518.7 -> 520.6 mm
