File: kicad/chouchou.kicad_pcb (KiCad board)
At the start: 2 copper layers, 261 x 90.8 mm, 84 parts

Commit message: add logo
Parts:
- added ?: LOGO, images:mushi, F.Cu at (67.4, 83.8)
- added ?: LOGO, images:mushi, F.Cu at (226.1, 83.8)
Routing:
- net mirror_matrix_pinky_bottom: track 127.3 -> 136.8 mm
- net matrix_pinky_bottom: track 144.4 -> 153.3 mm
- net matrix_ring_bottom: track 120.0 -> 123.0 mm
- net mirror_matrix_ring_bottom: track 103.4 -> 106.2 mm
- net matrix_middle_bottom: track 98.7 -> 100.1 mm
